File: pcb/n2k_meteo_gps_s3_tht/n2k_meteo_gps_s3_tht.kicad_sch (KiCad schematic)
At the start: 34 parts, among them U1 MCP2562-E-P, U2 ESP32-S3_SUPERMINI, U3 PC817, U5 TSR_1-2450, U6 TSR1-2433E

Commit message: PCB
Connections:
- net at U2.10 (GPIO10): now also J_BMP1.3 (Pin_3), J_I2C1.3 (Pin_3); no longer J_AUX1.3 (Pin_3)
- net at J_BMP1.4 (Pin_4), J_I2C1.4 (Pin_4): now also U2.9 (GPIO9); no longer U2.11 (GPIO11)
- net at U2.13 (GPIO13): now also U1.4 (RXD)
- net at U1.1 (TXD): now also U2.12 (GPIO12); no longer U2.7 (GPIO7)
- net at U2.8 (GPIO8): now also J_AUX1.3 (Pin_3); no longer U1.4 (RXD)
- net at J_AUX1.4 (Pin_4): now also U2.7 (GPIO7); no longer U2.9 (GPIO9)
Changed lines of the file:
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@@
-	(wire
-		(pts
-			(xy 111.76 109.22) (xy 156.21 109.22)
-		)
-		(stroke
-			(width 0)
-			(type default)
-		)
-	)
 	(wire
 		(pts
@@
 	(wire
 		(pts
+			(xy 127 99.06) (xy 127 81.28)
+		)
+		(stroke
+			(width 0)
+			(type default)
+		)
+	)
+	(wire
+		(pts
 			(xy 151.13 58.42) (xy 153.67 58.42)
 		)
@@
 	(wire
 		(pts
-			(xy 170.18 104.14) (xy 170.18 111.76)
+			(xy 170.18 104.14) (xy 170.18 106.68)
 		)
 		(stroke
@@
 	(wire
 		(pts
+			(xy 111.76 104.14) (xy 156.21 104.14)
+		)
+		(stroke
+			(width 0)
+			(type default)
+		)
+	)
+	(wire
+		(pts
 			(xy 190.5 36.83) (xy 190.5 55.88)
 		)
@@
 	(wire
 		(pts
-			(xy 127 104.14) (xy 127 81.28)
-		)
-		(stroke
-			(width 0)
-			(type default)
-		)
-	)
-	(wire
-		(pts
 			(xy 52.07 111.76) (xy 53.34 111.76)
 		)
@@
 	(wire
 		(pts
-			(xy 129.54 78.74) (xy 129.54 106.68)
+			(xy 129.54 78.74) (xy 129.54 101.6)
 		)
 		(stroke
@@
 	(wire
 		(pts
-			(xy 111.76 99.06) (xy 130.81 99.06)
-		)
-		(stroke
-			(width 0)
-			(type default)
-		)
-	)
-	(wire
-		(pts
 			(xy 175.26 82.55) (xy 173.99 82.55)
 		)
@@
 	(wire
 		(pts
-			(xy 73.66 125.73) (xy 130.81 125.73)
+			(xy 73.66 125.73) (xy 142.24 125.73)
 		)
 		(stroke
@@
 	(wire
 		(pts
-			(xy 130.81 125.73) (xy 130.81 114.3)
+			(xy 142.24 125.73) (xy 142.24 114.3)
 		)
 		(stroke
@@
 	(wire
 		(pts
-			(xy 132.08 50.8) (xy 132.08 101.6)
+			(xy 132.08 50.8) (xy 132.08 114.3)
 		)
 		(stroke
@@
 	(wire
 		(pts
+			(xy 111.76 114.3) (xy 132.08 114.3)
+		)
+		(stroke
+			(width 0)
+			(type default)
+		)
+	)
+	(wire
+		(pts
 			(xy 29.21 101.6) (xy 76.2 101.6)
 		)
@@
 	(wire
 		(pts
+			(xy 111.76 101.6) (xy 129.54 101.6)
+		)
+		(stroke
+			(width 0)
+			(type default)
+		)
+	)
+	(wire
+		(pts
 			(xy 69.85 144.78) (xy 129.54 144.78)
 		)
@@
 	(wire
 		(pts
+			(xy 111.76 99.06) (xy 127 99.06)
+		)
+		(stroke
+			(width 0)
+			(type default)
+		)
+	)
+	(wire
+		(pts
 			(xy 190.5 68.58) (xy 190.5 72.39)
 		)
@@
 	(wire
 		(pts
-			(xy 156.21 101.6) (xy 156.21 109.22)
+			(xy 156.21 101.6) (xy 156.21 104.14)
 		)
 		(stroke
@@
 	(wire
 		(pts
-			(xy 130.81 48.26) (xy 130.81 99.06)
+			(xy 130.81 48.26) (xy 130.81 111.76)
 		)
 		(stroke
@@
 	(wire
 		(pts
-			(xy 111.76 106.68) (xy 129.54 106.68)
-		)
-		(stroke
-			(width 0)
-			(type default)
-		)
-	)
-	(wire
-		(pts
 			(xy 194.31 156.21) (xy 226.06 156.21)
 		)
@@
 	(wire
 		(pts
-			(xy 170.18 111.76) (xy 111.76 111.76)
-		)
-		(stroke
-			(width 0)
-			(type default)
-		)
-	)
-	(wire
-		(pts
 			(xy 55.88 172.72) (xy 49.53 172.72)
 		)
@@
 	(wire
 		(pts
-			(xy 130.81 114.3) (xy 217.17 114.3)
+			(xy 142.24 114.3) (xy 217.17 114.3)
 		)
 		(stroke
@@
 	(wire
 		(pts
-			(xy 111.76 104.14) (xy 127 104.14)
-		)
-		(stroke
-			(width 0)
-			(type default)
-		)
-	)
-	(wire
-		(pts
 			(xy 60.96 45.72) (xy 63.5 45.72)
 		)
@@
 	(wire
 		(pts
+			(xy 111.76 106.68) (xy 170.18 106.68)
+		)
+		(stroke
+			(width 0)
+			(type default)
+		)
+	)
+	(wire
+		(pts
 			(xy 233.68 83.82) (xy 227.33 83.82)
 		)
@@
 	(wire
 		(pts
-			(xy 111.76 101.6) (xy 132.08 101.6)
-		)
-		(stroke
-			(width 0)
-			(type default)
-		)
-	)
-	(wire
-		(pts
 			(xy 119.38 87.63) (xy 119.38 93.98)
 		)
@@
 		)
 		(stroke
+			(width 0)
+			(type default)
+		)
+	)
+	(wire
+		(pts
+			(xy 111.76 111.76) (xy 130.81 111.76)
+		)
+		(stroke
