File: pcb/n2k_meteo_gps_s3_tht/n2k_meteo_gps_s3_tht_v0_aisler.kicad_pcb (KiCad board)
At the start: 2 copper layers, 59 x 68 mm, 34 parts, among them U1 MCP2562-E-P, U2 ESP32-S3_SUPERMINI, U3 PC817, U5 TSR_1-2450, U6 TSR1-2433E

Commit message: PCB
Parts:
- added R11: 4K7, Resistor_THT:R_Axial_DIN0207_L6.3mm_D2.5mm_P7.62mm_Horizontal, F.Cu at (31.6, 54.7)
- R10: value 2K -> 10K
- moved C4 8.00 mm to (27.1, 50.2), turned to 90 degrees
- moved R2 5.62 mm to (39.8, 37.6), turned to 90 degrees
Connections:
- C4 pad 1: Net-(D2--) -> Net-(D2-+)
- C4 pad 2: Net-(D2-+) -> Net-(D2--)
- J_T1 pad 1: +3.3V -> +5V
- R10 pad 2: Net-(D2-+) -> Net-(D2--)
- R2 pad 1: Net-(U2-GPIO3) -> GND
- R2 pad 2: GND -> Net-(U2-GPIO3)
- U2 pad 10: Net-(J_BMP1-Pin_3) -> Net-(J_AUX1-Pin_3)
- U2 pad 11: unconnected-(U2-GPIO11-Pad11) -> Net-(J_BMP1-Pin_4)
- U2 pad 12: Net-(U1-TXD) -> Net-(J_BMP1-Pin_3)
- U2 pad 13: Net-(U1-RXD) -> unconnected-(U2-GPIO13-Pad13)
- U2 pad 7: Net-(J_AUX1-Pin_4) -> Net-(U1-TXD)
- U2 pad 8: Net-(J_AUX1-Pin_3) -> Net-(U1-RXD)
- U2 pad 9: Net-(J_BMP1-Pin_4) -> Net-(J_AUX1-Pin_4)
- U3 pad 2: Net-(D2--) -> Net-(D2-+)
Routing:
- net Net-(R10-Pad1): track 10.0 -> 23.8 mm
- net Net-(D2-+): track 22.8 -> 34.9 mm
- net Net-(U1-RXD): track 38.4 -> 26.4 mm
- net Net-(U1-TXD): track 32.9 -> 23.2 mm
- net +3.3V: track 114.6 -> 108.1 mm
- net Net-(J_AUX1-Pin_4): track 10.4 -> 16.4 mm
- net Net-(J_AUX1-Pin_3): track 13.8 -> 19.0 mm
- net +5V: track 91.3 -> 93.9 mm
- net Net-(J_BMP1-Pin_4): track 17.2 -> 14.6 mm
- net Net-(D2--): track 27.2 -> 28.9 mm
- net Net-(U2-GPIO3): track 20.9 -> 22.2 mm
