File: pcb/n2k_meteo_gps_s3_tht/n2k_meteo_gps_s3_tht.kicad_pcb (KiCad board)
At the start: 2 copper layers, 59 x 74.8 mm, 45 parts, among them U1 MCP2562-E-P, U2 ESP32-S3_SUPERMINI, U3 PC817, U4 74AHC1G14, U5 LM7805_TO220, U6 TSR1-2433E

Commit message: Replaced MCP2562 PDIP-8 with SOIC-8 version. Tuned platformio.ini.
Parts:
- removed U1: MCP2562-E-P, Package_DIP:DIP-8_W7.62mm
- added U7: MCP2562-E-SN, Package_SO:SOIC-8_3.9x4.9mm_P1.27mm, F.Cu at (49.0, 76.5)
- C1, C7, C8: footprint Capacitor_THT:CP_Radial_Tantal_D4.5mm_P5.00mm -> Capacitor_THT:CP_Radial_Tantal_D5.0mm_P2.50mm
- moved C7 7.95 mm to (38.8, 61.5), turned to 180 degrees
- moved R1 7.60 mm to (48.3, 57.8), turned to 90 degrees
- moved C3 6.54 mm to (50.5, 68.8), turned to 90 degrees
- moved C8 5.25 mm to (41.0, 68.5)
- turned C6 to 90 degrees
Connections:
- D4 pad 1: Net-(J_CAN1-Pin_1) -> Net-(J_N2K1-Pin_1)
- D4 pad 2: Net-(J_N2K1-Pin_1) -> Net-(J_CAN1-Pin_1)
Routing:
- net Net-(J_LED1-Pin_1): track 39.4 -> 67.1 mm
- net Net-(J_N2K1-Pin_1): track 41.4 -> 58.0 mm
- net +3.3V: track 175.7 -> 165.5 mm
- net +5V: track 135.3 -> 144.5 mm
- net Net-(J_CAN1-Pin_1): track 48.8 -> 57.9 mm
- net Net-(D1-A): track 10.6 -> 7.51 mm
- net Net-(U2-GPIO13): track 52.2 -> 49.3 mm
- net Net-(U2-GPIO6): track 7.60 -> 5.04 mm
- net Net-(U2-GPIO12): track 49.9 -> 51.3 mm
