File: pcb/n2k_meteo_gps_s3_tht_v2.0_prod_06_2026/n2k_meteo_gps_s3_tht_prod_06_2026.kicad_pcb (KiCad board)
At the start: 2 copper layers, 59 x 74.8 mm, 45 parts, among them U1 MCP2562-E-P, U2 ESP32-S3_SUPERMINI, U3 PC817, U4 74AHC1G14, U5 LM7805_TO220, U6 TSR1-2433E

Commit message: updated pcb
Parts:
- C4: value 10nF -> 100nF
- R1: value 220Ω -> 100Ω
- R6: value 10K -> 12K
- U5: value LM7805_TO220 -> TSR_1-2450; footprint Package_TO_SOT_THT:TO-220-3_Vertical -> Converter_DCDC:Converter_DCDC_TRACO_TSR-1_THT
- moved D1 2.81 mm to (55.0, 59.8), turned to 0 degrees
Connections:
- C4 pad 1: Net-(D2-A) -> Net-(D3-A1)
- C4 pad 2: Net-(D2-K) -> Net-(D2-A)
- D1 pad 1: GND -> Net-(D1-K)
- D1 pad 2: Net-(D1-A) -> GND
- D3 pad 1: Net-(D2-A) -> Net-(D3-A1)
- J_ALT_G1 pad 1: Net-(D2-A) -> Net-(D3-A1)
- R1 pad 1: Net-(D1-A) -> Net-(D1-K)
- U3 pad 2: Net-(D2-A) -> Net-(D3-A1)
Routing:
- net Net-(D2-A): track 31.9 -> 4.89 mm
- net Net-(D3-A1): track 0.00 -> 24.1 mm
- net Net-(D1-K): track 0.00 -> 10.6 mm
- net Net-(D1-A): track 10.6 -> 0.00 mm
- net Net-(D2-K): track 55.6 -> 45.2 mm
- net Net-(J_CAN1-Pin_1): track 48.8 -> 48.1 mm
